File: hardware/veritas.kicad_sch (KiCad schematic)
At the start: 66 parts, among them J1 DISPLAY_PWR, J10 SYNC, J11 DEBUG, J12 CONTROLLER_PORT, J2 DISPLAY0, J3 DISPLAY1, J4 DISPLAY2, J5 DISPLAY3, J6 CON_RESET, J7 USB2.0_C, J8 VIDEO, J9 VIDEO, Q1 LMBT3946DW1T1G, Q2 2N7002K, SW1 ~{BOOT_SEL}, U1 W25Q128JVSIQ, U2 NCP1117ST33T3G, U3 RP2040, U4 MCP2221A, U5 LM1881, U6 TXS0108EPW, U7 TXS0108EPW, U8 TXS0108EPW, Y1 12MHz

Commit message: Completed new PCB revision. Includes different voltage translation and removal of unnecessary parts.
Parts:
- removed C17, C19: 0.1uF, Capacitor_SMD:C_0603_1608Metric_Pad1.08x0.95mm_HandSolder, symbol Device:C_Small
- removed JP1, JP2, JP5, JP6: SolderJumper_2_Open, Jumper:SolderJumper-2_P1.3mm_Open_TrianglePad1.0x1.5mm, symbol Jumper:SolderJumper_2_Open
- removed JP3: DJ-, Jumper:SolderJumper-3_P1.3mm_Open_RoundedPad1.0x1.5mm_NumberLabels, symbol Jumper:Jumper_3_Open
- removed JP4: DJ+, Jumper:SolderJumper-3_P1.3mm_Open_RoundedPad1.0x1.5mm_NumberLabels, symbol Jumper:Jumper_3_Open
- removed R4, R5: 1K, Resistor_SMD:R_0603_1608Metric_Pad0.98x0.95mm_HandSolder, symbol Device:R
- removed U4: MCP2221A, Package_DIP:DIP-14_W7.62mm, symbol veritas:MCP2221A
- removed U6, U7, U8: TXS0108EPW, Package_SO:TSSOP-20_4.4x6.5mm_P0.65mm, symbol Logic_LevelTranslator:TXS0108EPW
- added Q10, Q11, Q12, Q13, Q14, Q15, Q16, Q17, Q18, Q19, Q2, Q3, Q4, Q5, Q6, Q7, Q8, Q9: 2N7002K, Package_TO_SOT_SMD:SOT-23_Handsoldering, symbol Transistor_FET:2N7002K
- added R10, R11, R13, R14, R15, R16, R17, R18, R19, R20, R21, R23, R24, R25, R26, R27, R28, R29, R30, R31, R32, R33, R34, R35, R36, R37, R38, R39, R40, R41, R42, R43, R44, R46, R8, R9: 10K, Resistor_SMD:R_0603_1608Metric_Pad0.98x0.95mm_HandSolder, symbol Device:R_Small
- added U5, U6: SN74LVC1T45DRL, Package_TO_SOT_SMD:SOT-563, symbol Logic_LevelTranslator:SN74LVC1T45DRL
- J12: renamed from J11; footprint Connector_PinHeader_2.54mm:PinHeader_1x06_P2.54mm_Horizontal -> Connector_PinHeader_2.54mm:PinHeader_1x04_P2.54mm_Horizontal; symbol Connector_Generic:Conn_01x06 -> Connector_Generic:Conn_01x04
- renumbered C18 to C17, C20 to C18, C21 to C19, C22 to C20, C23 to C21, J12 to J11, JP7 to JP1, Q2 to Q20, R11 to R22, R6 to R4, R10 to R45, R7 to R5, R8 to R6, R9 to R7, U5 to U4
Connections:
- net BRIDGE_RX is gone; now on net CNT_0: U3.11 (GPIO8)
- net BRIDGE_TX is gone; now on net CNT_1: U3.12 (GPIO9)
- net PORTD+ is gone; now on net D+: J7.A6 (D+), J7.B6 (D+)
- net PORTD- is gone; now on net D-: J7.A7 (D-), J7.B7 (D-)
- net +3V3: now also Q10.1 (G), Q11.1 (G), Q12.1 (G), Q13.1 (G), Q14.1 (G), Q15.1 (G), Q16.1 (G), Q17.1 (G), Q18.1 (G), Q19.1 (G), Q2.1 (G), Q3.1 (G), Q4.1 (G), Q5.1 (G), Q6.1 (G), Q7.1 (G), Q8.1 (G), Q9.1 (G), R10.2, R14.2, R15.2, R16.2, R20.2, R21.2, R25.2, R26.2, R29.2, R30.2, R33.2, R34.2, R37.2, R38.2, R41.2, R42.2, R8.2, R9.2, U5.1 (VCCA), U6.1 (VCCA)
- net ALT_CLK_A: now also U3.9 (GPIO7); no longer U3.14 (GPIO11)
- net ALT_CLK_B: now also R46.1; no longer R12.1
- net CNT_0: now also Q7.2 (S), R16.1; no longer U3.15 (GPIO12)
- net CNT_1: now also Q4.2 (S), R10.1; no longer U3.16 (GPIO13)
- net CNT_10: now also U3.29 (GPIO18), Q18.2 (S), R41.1; no longer U3.34 (GPIO22)
- net CNT_11: now also U3.30 (GPIO19), Q16.2 (S), R37.1; no longer U3.35 (GPIO23)
- net CNT_12: now also U3.31 (GPIO20), Q14.2 (S), R33.1; no longer U3.36 (GPIO24)
- net CNT_13: now also U3.32 (GPIO21), Q12.2 (S), R29.1; no longer U3.37 (GPIO25)
- net CNT_14: now also U3.34 (GPIO22), Q10.2 (S), R25.1; no longer U3.38 (GPIO26_ADC0)
- net CNT_15: now also U3.35 (GPIO23), Q8.2 (S), R20.1; no longer U3.39 (GPIO27_ADC1)
- net CNT_16: now also U3.36 (GPIO24), Q5.2 (S), R14.1; no longer U3.40 (GPIO28_ADC2)
- net CNT_17: now also U3.37 (GPIO25), U5.3 (A); no longer J12.3 (Pin_3), U3.2 (GPIO0)
- net CNT_18: now also U3.38 (GPIO26_ADC0), U6.3 (A); no longer J12.2 (Pin_2), U3.3 (GPIO1)
- net CNT_2: now also U3.13 (GPIO10), Q19.2 (S), R42.1; no longer U3.17 (GPIO14)
- net CNT_3: now also U3.14 (GPIO11), Q17.2 (S), R38.1; no longer U3.18 (GPIO15)
- net CNT_4: now also U3.15 (GPIO12), Q15.2 (S), R34.1; no longer U3.27 (GPIO16)
- net CNT_5: now also U3.16 (GPIO13), Q13.2 (S), R30.1; no longer U3.28 (GPIO17)
- net CNT_6: now also U3.17 (GPIO14), Q11.2 (S), R26.1; no longer U3.29 (GPIO18)
- net CNT_7: now also U3.18 (GPIO15), Q9.2 (S), R21.1; no longer U3.30 (GPIO19)
- net CNT_8: now also U3.27 (GPIO16), Q6.2 (S), R15.1; no longer U3.31 (GPIO20)
- net CNT_9: now also U3.28 (GPIO17), Q3.2 (S), R9.1; no longer U3.32 (GPIO21)
- net CON_RESET: now also Q1.2 (B1), Q1.5 (B2), U3.8 (GPIO6); no longer U3.13 (GPIO10)
- net CP_1: now also U5.4 (B)
- net CP_11: now also U6.4 (B)
- net CP_13: now also Q10.3 (D), R27.1
- net CP_14: now also Q14.3 (D), R35.1
- net CP_15: now also Q18.3 (D), R43.1
- net CP_16: now also Q11.3 (D), R28.1
- net CP_17: now also Q15.3 (D), R36.1
- net CP_18: now also Q17.3 (D), R40.1
- net CP_21: now also Q8.3 (D), R23.1
- net CP_22: now also Q6.3 (D), R18.1
- net CP_23: now also Q7.3 (D), R19.1
- net CP_24: now also Q4.3 (D), R13.1
- net CP_25: now also Q19.3 (D), R44.1
- net CP_3: now also Q5.3 (D), R17.1
- net CP_4: now also Q12.3 (D), R31.1
- net CP_5: now also Q16.3 (D), R39.1
- net CP_6: now also R12.1, Q3.3 (D)
- net CP_7: now also Q9.3 (D), R24.1
- net CP_8: now also Q13.3 (D), R32.1
- net DETECT: now also Q2.2 (S), R8.1
- net DISPLAY_CLK: now also U3.7 (GPIO5); no longer U3.9 (GPIO7)
- net DISPLAY_SER: now also U3.6 (GPIO4); no longer U3.8 (GPIO6)
- net DISPLAY_STROBE0: now also U3.2 (GPIO0); no longer U3.4 (GPIO2)
- net DISPLAY_STROBE1: now also U3.3 (GPIO1); no longer U3.5 (GPIO3)
- net DISPLAY_STROBE2: now also U3.4 (GPIO2); no longer U3.6 (GPIO4)
- net DISPLAY_STROBE3: now also U3.5 (GPIO3); no longer U3.7 (GPIO5)
- net GND: now also J12.4 (Pin_4), U5.2 (GND), U6.2 (GND); no longer J12.6 (Pin_6)
- net SWCLK: now also J12.2 (Pin_2); no longer J12.4 (Pin_4)
- net SWD: now also J12.3 (Pin_3); no longer J12.5 (Pin_5)
- net VBUS: now also R46.2; no longer R12.2
- net CP_20 renamed SYSTEM_PWR
- net SYSTEM_PWR: now also R12.2, R11.2, R13.2, R17.2, R18.2, R19.2, R23.2, R24.2, R27.2, R28.2, R31.2, R32.2, R35.2, R36.2, R39.2, R40.2, R43.2, R44.2, U5.6 (VCCB), U6.6 (VCCB)
- new net: Q2.3 (D), R11.1
- new net CNT_17_DIR: U3.39 (GPIO27_ADC1), U5.5 (DIR)
- new net CNT_18_DIR: U3.40 (GPIO28_ADC2), U6.5 (DIR)
- no-connect marks 17 -> 4
Other:
- note removed: "CP_20 is used for DETECT (translated) and SYSTEM_PWR"
- moved on the sheet: C20, C21, J11, JP1, Q20, R45
