File: hardware/veritas.kicad_sch (KiCad schematic)
At the start: 108 parts, among them J1 DISPLAY_PWR, J10 SYNC, J11 CONTROLLER_PORT, J12 DEBUG, J2 DISPLAY0, J3 DISPLAY1, J4 DISPLAY2, J5 DISPLAY3, J6 CON_RESET, J7 USB2.0_C, J8 VIDEO, J9 VIDEO, Q1 LMBT3946DW1T1G, Q10 2N7002K, Q11 2N7002K, Q12 2N7002K, Q13 2N7002K, Q14 2N7002K, Q15 2N7002K, Q16 2N7002K, Q17 2N7002K, Q18 2N7002K, Q19 2N7002K, Q2 2N7002K, Q20 2N7002K, Q3 2N7002K, Q4 2N7002K, Q5 2N7002K, Q6 2N7002K, Q7 2N7002K, Q8 2N7002K, Q9 2N7002K, SW1 ~{BOOT_SEL}, U1 W25Q128JVSIQ, U2 NCP1117ST33T3G, U3 RP2040, U4 LM1881, U5 SN74LVC1T45DRL, U6 SN74LVC1T45DRL, Y1 12MHz

Commit message: Produced new version as of 2023-05-07: - Replaced reset circuit with TTL-compatible buffer IC (untested; uses /OE to isolate signal from console until reset is activated) - Set more components to be assembled by manufacturer - Replaced THT crystal with SMD variant - Added /RESET pushbutton - Fixed incorrect layout for the two high-speed translation/buffer channels
Parts:
- removed Q1: LMBT3946DW1T1G, Package_TO_SOT_SMD:SOT-363_SC-70-6_Handsoldering, symbol Transistor_BJT:FFB3946
- added R3: 10K, Resistor_SMD:R_0603_1608Metric_Pad0.98x0.95mm_HandSolder, symbol Device:R_Small
- added SW2: ~{RESET}, Button_Switch_SMD:SW_SPST_PTS645, symbol Switch:SW_Push
- added U4: 74LVC2G240, Package_SO:TSSOP-8_3x3mm_P0.65mm, symbol veritas:74LVC2G240
- U6: renamed from U5; footprint Package_TO_SOT_SMD:SOT-563 -> Package_TO_SOT_SMD:SOT-363_SC-70-6
- U7: renamed from U6; footprint Package_TO_SOT_SMD:SOT-563 -> Package_TO_SOT_SMD:SOT-363_SC-70-6
- Y1: footprint Crystal:Crystal_SMD_HC49-SD -> Crystal:Crystal_SMD_3225-4Pin_3.2x2.5mm; symbol Device:Crystal -> Device:Crystal_GND24
- renumbered Q2 to Q1, Q11 to Q10, Q12 to Q11, Q13 to Q12, Q14 to Q13, Q15 to Q14, Q16 to Q15, Q17 to Q16, Q18 to Q17, Q19 to Q18, Q20 to Q19, Q3 to Q2, Q4 to Q3, Q5 to Q4, Q6 to Q5, Q7 to Q6, Q8 to Q7, Q9 to Q8, Q10 to Q9, R9 to R10, R10 to R11, R11 to R12, R12 to R13, R13 to R14, R14 to R15, R15 to R16, R16 to R17, R17 to R18, R18 to R19, R19 to R20, R20 to R21, R21 to R22, R22 to R23, R23 to R24, R24 to R25, R25 to R26, R26 to R27, R27 to R28, R28 to R29, R29 to R30, R30 to R31, R31 to R32, R32 to R33, R33 to R34, R34 to R35, R35 to R36, R36 to R37, R37 to R38, R38 to R39, R3 to R4, R39 to R40, R40 to R41, R41 to R42, R42 to R43, R43 to R44, R44 to R45, R45 to R46, R46 to R47, R4 to R5, R5 to R6, R6 to R7, R7 to R8, R8 to R9, U4 to U5
Connections:
- net +3V3: now also R3.2; no longer U3.26 (RUN)
- net GND: now also Y1.2, Y1.4, SW2.1, U4.4 (GND), U4.5 (2A)
- net RESET_HI: now also U4.3 (2Y)
- net RESET_LO: now also U4.6 (1Y)
- net SYSTEM_PWR: now also U4.2 (1A), U4.8 (VCC)
- net at C13.2, U3.20 (XIN): now also Y1.3; no longer Y1.2
- net CON_RESET renamed ~{CON_RESET}
- net ~{CON_RESET}: now also U4.1 (1~{OE}), U4.7 (2~{OE})
- new net: R3.1, SW2.2, U3.26 (RUN)
Other:
- moved on the sheet: C13, C14, J6, R4
