File: hardware/veritas.kicad_pcb (KiCad board)
At the start: 2 copper layers, 76.1 x 77.3 mm, 112 parts, among them J1 DISPLAY_PWR, J10 SYNC, J11 CONTROLLER_PORT, J12 DEBUG, J2 DISPLAY0, J3 DISPLAY1, J4 DISPLAY2, J5 DISPLAY3, J6 CON_RESET, J7 USB2.0_C, J8 VIDEO, J9 VIDEO, Q1 LMBT3946DW1T1G, Q10 2N7002K, Q11 2N7002K, Q12 2N7002K, Q13 2N7002K, Q14 2N7002K, Q15 2N7002K, Q16 2N7002K, Q17 2N7002K, Q18 2N7002K, Q19 2N7002K, Q2 2N7002K, Q20 2N7002K, Q3 2N7002K, Q4 2N7002K, Q5 2N7002K, Q6 2N7002K, Q7 2N7002K, Q8 2N7002K, Q9 2N7002K, SW1 ~{BOOT_SEL}, U1 W25Q128JVSIQ, U2 NCP1117ST33T3G, U3 RP2040, U4 LM1881, U5 SN74LVC1T45DRL, U6 SN74LVC1T45DRL, Y1 12MHz

Commit message: Produced new version as of 2023-05-07: - Replaced reset circuit with TTL-compatible buffer IC (untested; uses /OE to isolate signal from console until reset is activated) - Set more components to be assembled by manufacturer - Replaced THT crystal with SMD variant - Added /RESET pushbutton - Fixed incorrect layout for the two high-speed translation/buffer channels
Parts:
- removed the Q1 at (127.3, 84.0)
- added R3: 10K, Resistor_SMD:R_0603_1608Metric_Pad0.98x0.95mm_HandSolder, F.Cu at (154.7, 95.6)
- added SW2: ~{RESET}, Button_Switch_SMD:SW_SPST_PTS645, F.Cu at (170.5, 79.2)
- added U4: 74LVC2G240, Package_SO:TSSOP-8_3x3mm_P0.65mm, F.Cu at (125.2, 84.7)
- U6: renamed from U5; footprint Package_TO_SOT_SMD:SOT-563 -> Package_TO_SOT_SMD:SOT-363_SC-70-6
- U7: renamed from U6; footprint Package_TO_SOT_SMD:SOT-563 -> Package_TO_SOT_SMD:SOT-363_SC-70-6
- Y1: footprint Crystal:Crystal_SMD_HC49-SD -> Crystal:Crystal_SMD_3225-4Pin_3.2x2.5mm
- moved C14 4.61 mm to (128.0, 96.5), turned to 0 degrees
- moved C13 4.43 mm to (125.5, 93.3)
- moved SW1 2.54 mm to (159.9, 79.2)
- moved Y1 1.12 mm to (128.1, 93.6)
- moved U7 0.44 mm to (161.4, 100.5)
- moved U6 0.19 mm to (164.3, 100.5)
- renumbered Q2 to Q1, Q11 to Q10, Q12 to Q11, Q13 to Q12, Q14 to Q13, Q15 to Q14, Q16 to Q15, Q17 to Q16, Q18 to Q17, Q19 to Q18, Q20 to Q19, Q3 to Q2, Q4 to Q3, Q5 to Q4, Q6 to Q5, Q7 to Q6, Q8 to Q7, Q9 to Q8, Q10 to Q9, R9 to R10, R10 to R11, R11 to R12, R12 to R13, R13 to R14, R14 to R15, R15 to R16, R16 to R17, R17 to R18, R18 to R19, R19 to R20, R20 to R21, R21 to R22, R22 to R23, R23 to R24, R24 to R25, R25 to R26, R26 to R27, R27 to R28, R28 to R29, R29 to R30, R30 to R31, R31 to R32, R32 to R33, R33 to R34, R34 to R35, R35 to R36, R36 to R37, R37 to R38, R38 to R39, R3 to R4, R39 to R40, R40 to R41, R41 to R42, R42 to R43, R43 to R44, R44 to R45, R45 to R46, R46 to R47, R4 to R5, R5 to R6, R6 to R7, R7 to R8, R8 to R9, U4 to U5
Connections:
- C13 pad 2: Net-(C13-Pad2) -> Net-(U3-XIN)
- U3 pad 20: Net-(C13-Pad2) -> Net-(U3-XIN)
- U3 pad 26: +3V3 -> Net-(U3-RUN)
- U3 pad 8: CON_RESET -> ~{CON_RESET}
- Y1 pad 2: Net-(C13-Pad2) -> GND
Routing:
- net Net-(U3-RUN): track 0.00 -> 63.5 mm, vias 0 -> 4
- net ~{CON_RESET}: track 0.00 -> 24.0 mm, vias 0 -> 2
- net GND: track 134.6 -> 155.3 mm, vias 27 -> 26
- net CON_RESET: track 20.4 -> 0.00 mm
- net Net-(C13-Pad2): track 16.3 -> 0.00 mm
- net Net-(U3-XIN): track 0.00 -> 12.3 mm
- net Net-(C14-Pad2): track 11.9 -> 5.13 mm
- net ALT_CLK_A: track 42.2 -> 37.5 mm
- net /RESET_HI: track 9.14 -> 6.12 mm, vias 1 -> 0
- net Net-(R1-Pad1): track 12.6 -> 10.1 mm
- net SYSTEM_PWR: track 205.7 -> 206.7 mm
- net +3V3: track 275.7 -> 276.6 mm
Other:
- board text added: "by Bigbass CERN-OHL-W-2.0 2023-05-07"
- board text removed: "by Bigbass CERN-OHL-W-2.0 2022-09-06"
